Commit message: added camera and imu sensors

File: description/robot.urdf.xacro (robot description, xacro)
@@ -2,3 +2,6 @@
 <robot xmlns:xacro="http://www.ros.org/wiki/xacro"  name="robot">
 <xacro:include filename="robot_core.xacro" />
+<xacro:include filename="gazebo_control.xacro" />
+<xacro:include filename="camera.xacro" />
+<xacro:include filename="imu.xacro" />
 </robot>

File: description/robot_core.xacro (robot description, xacro)
@@ -50,4 +50,7 @@
         </xacro:inertial_box>
     </link>
+    <gazebo reference="chassis">
+        <material>Gazebo/White</material>
+    </gazebo>
     <!-- (Left Wheel)
     adjusted the orientation of the cylinder made its axis of rotation z-->
@@ -74,4 +77,7 @@
         </xacro:inertial_cylinder>
     </link>
+    <gazebo reference="left_wheel">
+        <material>Gazebo/Blue</material>
+    </gazebo>
     <!-- (Right Wheel)
     same as left but opposite angle and axis of rotation-->
@@ -98,4 +104,7 @@
         </xacro:inertial_cylinder>
     </link>
+        <gazebo reference="right_wheel">
+        <material>Gazebo/Blue</material>
+    </gazebo>
     <!--(Caster Wheel)-->
     <joint name = "caster_wheel_joint" type = "fixed">
@@ -120,3 +129,8 @@
         </xacro:inertial_sphere>
     </link>
+<gazebo reference="caster_wheel">
+        <material>Gazebo/Black</material>
+        <mu1 value="0.001"/>
+        <mu2 value="0.001"/>
+    </gazebo>
 </robot>
